Commit message: Spawn multi rounded_shape robot

File: simulation_ws/src/robot_bringup/descriptions/robot_swarm.urdf (robot description, URDF)
Before this commit: robot robot, 6 links, 5 joints
Links:
- removed link caster_wheel
- added link back_caster_wheel, mass 0.1; collision sphere radius=0.03; visual sphere radius=0.03
- added link front_caster_wheel, mass 0.1; collision sphere radius=0.03; visual sphere radius=0.03
- link chassis: mass 0.5 -> 2.0; geometry collision cylinder length=0.15 radius=0.15; visual cylinder length=0.15 radius=0.15
- link laser_frame: mass 0.1 -> None; geometry visual cylinder length=0.035 radius=0.045
- link left_wheel: mass 0.1 -> 0.02; geometry collision cylinder length=0.03 radius=0.04; visual cylinder length=0.03 radius=0.04
- link right_wheel: mass 0.1 -> 0.02; geometry collision cylinder length=0.03 radius=0.04; visual cylinder length=0.03 radius=0.04
Joints:
- removed joint caster_wheel_joint
- added joint back_caster_wheel_joint: type fixed, parent chassis, child back_caster_wheel, origin xyz=-0.1 0 -0.063
- added joint front_caster_wheel_joint: type fixed, parent chassis, child front_caster_wheel, origin xyz=0.1 0 -0.0625555
- joint chassis_joint: origin xyz=-0.1 0 0 -> xyz=0 0 0
- joint laser_joint: origin xyz=0.1 0 0.175 rpy=0 0 0 -> xyz=0 0 0.085 rpy=0 0 0
- joint left_wheel_joint: origin xyz=0 0.175 0 rpy=-1.5707963267948966 0 0 -> xyz=0 0.14 -0.055 rpy=-1.57079632679 3.14159265358 0; parent base_link -> chassis
- joint right_wheel_joint: origin xyz=0 -0.175 0 rpy=1.5707963267948966 0 0 -> xyz=0 -0.14 -0.055 rpy=1.57079632679 0 0; parent base_link -> chassis
