Commit message: Construct file

File: simulation_ws/src/robot_bringup/descriptions/gazebo_control.xacro (robot description, xacro)
@@ -6,6 +6,6 @@
             <!-- ROS parameters -->
             <!-- <ros>
-            <namespace>robot_namespace</namespace>
-            <param name="robot_description" value="robot_description" />
+                <namespace>robot_namespace</namespace>
+                <param name="robot_description" value="robot_description" />
             </ros> -->
             <!-- Wheel Information -->

File: simulation_ws/src/robot_bringup/descriptions/lidar.xacro (robot description, xacro)
@@ -1,29 +1,32 @@
 <?xml version="1.0"?>
 <robot xmlns:xacro="http://www.ros.org/wiki/xacro" >
-    <joint name="laser_joint" type="fixed">
-        <parent link="chassis"/>
-        <child link="laser_frame"/>
-        <origin xyz="0.1 0 0.175" rpy="0 0 0"/>
-    </joint>
     <link name="laser_frame">
         <visual>
             <geometry>
-                <cylinder radius="0.05" length="0.04"/>
+                <cylinder radius="0.0325" length="0.045"/>
             </geometry>
-            <material name="red"/>
+            <material name="orange">
+                <color rgba="1 0.3 0.1 1"/>
+            </material>
         </visual>
         <collision>
             <geometry>
-                <cylinder radius="0.05" length="0.04"/>
+                <cylinder radius="0.0325" length="0.045"/>
             </geometry>
         </collision>
-        <xacro:inertial_cylinder mass="0.1" length="0.04" radius="0.05">
+        <xacro:inertial_cylinder mass="0.1" length="0.045" radius="0.0325">
             <origin xyz="0 0 0" rpy="0 0 0"/>
         </xacro:inertial_cylinder>
     </link>
+    <joint name="laser_joint" type="fixed">
+        <parent link="base_link"/>
+        <child link="laser_frame"/>
+        <origin xyz="0 0 0.205" rpy="0 0 0"/>
+    </joint>
     <gazebo reference="laser_frame">
-        <material>Gazebo/Red</material>
+        <material>Gazebo/Orange</material>
         <sensor name="laser" type="ray">
             <pose> 0 0 0 0 0 0 </pose>
+            <always_on>true</always_on>
             <visualize>true</visualize>
             <update_rate>10</update_rate>
@@ -32,5 +35,4 @@
                     <horizontal>
                         <samples>360</samples>
-                        <resolution>0.4</resolution>
                         <min_angle>-3.14</min_angle>
                         <max_angle>3.14</max_angle>
@@ -38,7 +40,6 @@
                 </scan>
                 <range>
-                    <min>0.3</min>
+                    <min>0.2</min>
                     <max>12</max>
-                    <resolution>0.01</resolution>
                 </range>
             </ray>
@@ -48,4 +49,5 @@
                 </ros>
                 <output_type>sensor_msgs/LaserScan</output_type>
+                <!-- <topicName>/scan</topicName> -->
                 <frame_name>laser_frame</frame_name>
             </plugin>
