Commit message: fix two passive wheels' positions

File: simulation_ws/src/description/swarm_bot.urdf (robot description, URDF)
Before this commit: robot swarm_bot, 6 links, 5 joints
Joints:
- joint back_passive_wheel_joint: origin xyz=-0.085 0 -0.065 rpy=0 0 0 -> xyz=-0.067 0 -0.071 rpy=0 0 0
- joint front_passive_wheel_joint: origin xyz=0.085 0 -0.065 rpy=0 0 0 -> xyz=0.067 0 -0.0735 rpy=0 0 0
