Commit message: Move the robot on the ground

File: simulation_ws/src/description/swarm_bot.urdf.xacro (robot description, xacro)
@@ -1,13 +1,15 @@
 <?xml version="1.0"?>
-<robot name="swarm_bot">
+<robot xmlns:xacro="http://www.ros.org/wiki/xacro"  name="swarm_bot">
     <!-- Base -->
     <link name="base_link">
         <visual>
+            <!-- change the position of the visualization only, not the axis -->
+            <origin xyz="0 0 0.1075" rpy="0 0 0"/>
             <geometry>
                 <!-- unit: meter -->
                 <cylinder radius="0.107" length="0.15"/>
             </geometry>
-            <material name="gray">
-                <color rgba="0.5 0.5 0.5 1.0"/>
+            <material name="white">
+                <color rgba="1 1 1 1"/>
             </material>
         </visual>
@@ -69,15 +71,17 @@
     </link>
     <!-- Joints -->
+    <!-- Left Wheel -->
     <joint name="left_wheel_joint" type="continuous">
         <parent link="base_link"/>
         <child link="left_wheel"/>
-        <!-- rotate wheel 90 deg around y-axis -->
-        <origin xyz="0 -0.107 -0.065" rpy="1.5708 0 0"/>
+        <!-- rotate wheel 90 deg around x-axis -->
+        <origin xyz="0 -0.107 0.0325" rpy="-1.5708 0 0"/>
         <axis xyz="0 1 0"/>
     </joint>
+    <!-- Right Wheel -->
     <joint name="right_wheel_joint" type="continuous">
         <parent link="base_link"/>
         <child link="right_wheel"/>
-        <origin xyz="0 0.107 -0.065" rpy="1.5708 0 0"/>
+        <origin xyz="0 0.107 0.0325" rpy="1.5708 0 0"/>
         <axis xyz="0 1 0"/>
     </joint>
@@ -86,5 +90,5 @@
         <parent link="base_link"/>
         <child link="front_passive_wheel"/>
-        <origin xyz="0.067 0 -0.0735" rpy="0 0 0"/>
+        <origin xyz="0.067 0 0.024" rpy="0 0 0"/>
     </joint>
     <!-- Back Passive Wheel -->
@@ -92,10 +96,11 @@
         <parent link="base_link"/>
         <child link="back_passive_wheel"/>
-        <origin xyz="-0.067 0 -0.071" rpy="0 0 0"/>
+        <origin xyz="-0.067 0 0.022" rpy="0 0 0"/>
     </joint>
+    <!-- Lidar -->
     <joint name="lidar_joint" type="fixed">
         <parent link="base_link"/>
         <child link="lidar"/>
-        <origin xyz="0 0 0.075" rpy="0 0 0"/>
+        <origin xyz="0 0 0.205" rpy="0 0 0"/>
     </joint>
 </robot>

Commit message: Add collision and inertia tags

File: simulation_ws/src/description/swarm_bot.urdf.xacro (robot description, xacro)
@@ -1,4 +1,5 @@
 <?xml version="1.0"?>
 <robot xmlns:xacro="http://www.ros.org/wiki/xacro"  name="swarm_bot">
+    <xacro:include filename="inertial_macros.xacro" />
     <!-- Base -->
     <link name="base_link">
@@ -14,4 +15,13 @@
             </material>
         </visual>
+        <collision>
+            <origin xyz="0 0 0.1075" rpy="0 0 0"/>
+            <geometry>
+                <cylinder radius="0.107" length="0.15"/>
+            </geometry>
+        </collision>
+        <xacro:inertial_cylinder mass="0.5" length="0.15" radius="0.107">
+            <origin xyz="0 0 0.1075" rpy="0 0 0"/>
+        </xacro:inertial_cylinder>
     </link>
     <!-- Left Wheel -->
@@ -25,4 +35,12 @@
             </material>
         </visual>
+        <collision>
+            <geometry>
+                <cylinder radius="0.0325" length="0.03"/>
+            </geometry>
+        </collision>
+        <xacro:inertial_cylinder mass="0.2" length="0.03" radius="0.0325">
+            <origin xyz="0 0 0" rpy="0 0 0"/>
+        </xacro:inertial_cylinder>
     </link>
     <!-- Right Wheel -->
@@ -36,4 +54,12 @@
             </material>
         </visual>
+        <collision>
+            <geometry>
+                <cylinder radius="0.0325" length="0.03"/>
+            </geometry>
+        </collision>
+        <xacro:inertial_cylinder mass="0.2" length="0.03" radius="0.0325">
+            <origin xyz="0 0 0" rpy="0 0 0"/>
+        </xacro:inertial_cylinder>
     </link>
     <!-- Front Passive Wheel -->
@@ -47,4 +73,12 @@
             </material>
         </visual>
+        <collision>
+            <geometry>
+                <sphere radius="0.024"/>
+            </geometry>
+        </collision>
+        <xacro:inertial_sphere mass="0.1" radius="0.05">
+            <origin xyz="0 0 0" rpy="0 0 0"/>
+        </xacro:inertial_sphere>
     </link>
     <!-- Back Passive Wheel -->
@@ -58,4 +92,12 @@
             </material>
         </visual>
+        <collision>
+            <geometry>
+                <sphere radius="0.024"/>
+            </geometry>
+        </collision>
+        <xacro:inertial_sphere mass="0.1" radius="0.024">
+            <origin xyz="0 0 0" rpy="0 0 0"/>
+        </xacro:inertial_sphere>
     </link>
     <!-- Lidar -->
@@ -69,4 +111,12 @@
             </material>
         </visual>
+        <collision>
+            <geometry>
+                <cylinder radius="0.0325" length="0.045"/>
+            </geometry>
+        </collision>
+        <xacro:inertial_cylinder mass="0.1" length="0.045" radius="0.0325">
+            <origin xyz="0 0 0" rpy="0 0 0"/>
+        </xacro:inertial_cylinder>
     </link>
     <!-- Joints -->
