Commit message: Adjust lidar

File: simulation_ws/src/navigation/description/lidar.xacro (robot description, xacro)
@@ -1,11 +1,11 @@
 <?xml version="1.0"?>
 <robot xmlns:xacro="http://www.ros.org/wiki/xacro" >
-    <link name="lidar">
+    <link name="laser_frame">
         <visual>
             <geometry>
                 <cylinder radius="0.0325" length="0.045"/>
             </geometry>
-            <material name="blue">
-                <color rgba="0.0 0.0 1.0 1.0"/>
+            <material name="orange">
+                <color rgba="1 0.3 0.1 1"/>
             </material>
         </visual>
@@ -19,13 +19,10 @@
         </xacro:inertial_cylinder>
     </link>
-    <gazebo reference="lidar">
-        <material>Gazebo/Blue</material>
-    </gazebo>
-    <joint name="lidar_joint" type="fixed">
-        <parent link="origin_link"/>
-        <child link="lidar"/>
-        <origin xyz="0 0 0.1725" rpy="0 0 0"/>
+    <joint name="laser_joint" type="fixed">
+        <parent link="base_link"/>
+        <child link="laser_frame"/>
+        <origin xyz="0 0 0.205" rpy="0 0 0"/>
     </joint>
-    <gazebo reference="lidar">
+    <gazebo reference="laser_frame">
         <material>Gazebo/Orange</material>
         <sensor name="laser" type="ray">
@@ -43,5 +40,5 @@
                 </scan>
                 <range>
-                    <min>0.3</min>
+                    <min>0.2</min>
                     <max>12</max>
                 </range>
@@ -52,4 +49,5 @@
                 </ros>
                 <output_type>sensor_msgs/LaserScan</output_type>
+                <!-- <topicName>/scan</topicName> -->
                 <frame_name>laser_frame</frame_name>
             </plugin>
