Commit message: Generate Gazebo control file

File: simulation_ws/src/navigation/description/swarm_bot.urdf.xacro (robot description, xacro)
@@ -2,4 +2,9 @@
 <robot xmlns:xacro="http://www.ros.org/wiki/xacro"  name="swarm_bot">
     <xacro:include filename="inertial_macros.xacro" />
+    <xacro:include filename="gazebo_control.xacro" />
+    <!-- LINKS -->
+    <!-- Origin -->
+    <link name="origin_link">
+    </link>
     <!-- Base -->
     <link name="base_link">
@@ -8,5 +13,5 @@
             <origin xyz="0 0 0.1075" rpy="0 0 0"/>
             <geometry>
-                <!-- unit: meter -->
+                <!-- unit/ meter -->
                 <cylinder radius="0.107" length="0.15"/>
             </geometry>
@@ -25,5 +30,5 @@
         </xacro:inertial_cylinder>
     </link>
-    <gazebo reference="base">
+    <gazebo reference="base_link">
         <material>Gazebo/White</material>
     </gazebo>
@@ -122,5 +127,5 @@
     </gazebo>
     <!-- Lidar -->
-    <link name="lidar">
+    <!-- <link name="lidar">
         <visual>
             <geometry>
@@ -142,38 +147,44 @@
     <gazebo reference="lidar">
         <material>Gazebo/Blue</material>
-    </gazebo>
-    <!-- Joints -->
+    </gazebo> -->
+    <!-- JOINTS-->
+    <!-- Base -->
+    <joint name="origin_joint" type="fixed">
+        <parent link="origin_link"/>
+        <child link="base_link"/>
+        <origin xyz="0 0 -0.0325"/>
+    </joint>
     <!-- Left Wheel -->
     <joint name="left_wheel_joint" type="continuous">
-        <parent link="base_link"/>
+        <parent link="origin_link"/>
         <child link="left_wheel"/>
         <!-- rotate wheel 90 deg around x-axis -->
-        <origin xyz="0 -0.107 0.0325" rpy="-1.5708 0 0"/>
-        <axis xyz="0 1 0"/>
+        <origin xyz="0 -0.107 0" rpy="-${pi/2} 0 0"/>
+        <axis xyz="0 0 1"/>
     </joint>
     <!-- Right Wheel -->
     <joint name="right_wheel_joint" type="continuous">
-        <parent link="base_link"/>
+        <parent link="origin_link"/>
         <child link="right_wheel"/>
-        <origin xyz="0 0.107 0.0325" rpy="1.5708 0 0"/>
-        <axis xyz="0 1 0"/>
+        <origin xyz="0 0.107 0" rpy="${pi/2} 0 0"/>
+        <axis xyz="0 0 -1"/>
     </joint>
     <!-- Front Passive Wheel -->
     <joint name="front_passive_wheel_joint" type="continuous">
-        <parent link="base_link"/>
+        <parent link="origin_link"/>
         <child link="front_passive_wheel"/>
-        <origin xyz="0.067 0 0.024" rpy="0 0 0"/>
+        <origin xyz="0.067 0 -0.0085" rpy="0 0 0"/>
     </joint>
     <!-- Back Passive Wheel -->
     <joint name="back_passive_wheel_joint" type="continuous">
-        <parent link="base_link"/>
+        <parent link="origin_link"/>
         <child link="back_passive_wheel"/>
-        <origin xyz="-0.067 0 0.022" rpy="0 0 0"/>
+        <origin xyz="-0.067 0 -0.0083" rpy="0 0 0"/>
     </joint>
     <!-- Lidar -->
-    <joint name="lidar_joint" type="fixed">
-        <parent link="base_link"/>
+    <!-- <joint name="lidar_joint" type="fixed">
+        <parent link="origin_link"/>
         <child link="lidar"/>
-        <origin xyz="0 0 0.205" rpy="0 0 0"/>
-    </joint>
+        <origin xyz="0 0 0.1725" rpy="0 0 0"/>
+    </joint> -->
 </robot>

Commit message: Add lidar

File: simulation_ws/src/navigation/description/swarm_bot.urdf.xacro (robot description, xacro)
@@ -3,4 +3,5 @@
     <xacro:include filename="inertial_macros.xacro" />
     <xacro:include filename="gazebo_control.xacro" />
+    <xacro:include filename="lidar.xacro" />
     <!-- LINKS -->
     <!-- Origin -->
@@ -126,26 +127,4 @@
         <mu2 value="0.001"/>
     </gazebo>
-    <!-- Lidar -->
-    <!-- <link name="lidar">
-        <visual>
-            <geometry>
-                <cylinder radius="0.0325" length="0.045"/>
-            </geometry>
-            <material name="blue">
-                <color rgba="0.0 0.0 1.0 1.0"/>
-            </material>
-        </visual>
-        <collision>
-            <geometry>
-                <cylinder radius="0.0325" length="0.045"/>
-            </geometry>
-        </collision>
-        <xacro:inertial_cylinder mass="0.1" length="0.045" radius="0.0325">
-            <origin xyz="0 0 0" rpy="0 0 0"/>
-        </xacro:inertial_cylinder>
-    </link>
-    <gazebo reference="lidar">
-        <material>Gazebo/Blue</material>
-    </gazebo> -->
     <!-- JOINTS-->
     <!-- Base -->
@@ -182,9 +161,3 @@
         <origin xyz="-0.067 0 -0.0083" rpy="0 0 0"/>
     </joint>
-    <!-- Lidar -->
-    <!-- <joint name="lidar_joint" type="fixed">
-        <parent link="origin_link"/>
-        <child link="lidar"/>
-        <origin xyz="0 0 0.1725" rpy="0 0 0"/>
-    </joint> -->
 </robot>

Commit message: add control robot files

File: simulation_ws/src/navigation/description/swarm_bot.urdf.xacro (robot description, xacro)
@@ -35,4 +35,26 @@
     </gazebo>
     <!-- Left Wheel -->
+    <link name="right_wheel">
+        <visual>
+            <geometry>
+                <cylinder radius="0.0325" length="0.03"/>
+            </geometry>
+            <material name="black">
+                <color rgba="0.0 0.0 0.0 1.0"/>
+            </material>
+        </visual>
+        <collision>
+            <geometry>
+                <cylinder radius="0.0325" length="0.03"/>
+            </geometry>
+        </collision>
+        <xacro:inertial_cylinder mass="0.2" length="0.03" radius="0.0325">
+            <origin xyz="0 0 0" rpy="0 0 0"/>
+        </xacro:inertial_cylinder>
+    </link>
+    <gazebo reference="right_wheel">
+        <material>Gazebo/Black</material>
+    </gazebo>
+    <!-- Right Wheel -->
     <link name="left_wheel">
         <visual>
@@ -54,26 +76,4 @@
     </link>
     <gazebo reference="left_wheel">
-        <material>Gazebo/Black</material>
-    </gazebo>
-    <!-- Right Wheel -->
-    <link name="right_wheel">
-        <visual>
-            <geometry>
-                <cylinder radius="0.0325" length="0.03"/>
-            </geometry>
-            <material name="black">
-                <color rgba="0.0 0.0 0.0 1.0"/>
-            </material>
-        </visual>
-        <collision>
-            <geometry>
-                <cylinder radius="0.0325" length="0.03"/>
-            </geometry>
-        </collision>
-        <xacro:inertial_cylinder mass="0.2" length="0.03" radius="0.0325">
-            <origin xyz="0 0 0" rpy="0 0 0"/>
-        </xacro:inertial_cylinder>
-    </link>
-    <gazebo reference="right_wheel">
         <material>Gazebo/Black</material>
     </gazebo>
@@ -135,7 +135,7 @@
     </joint>
     <!-- Left Wheel -->
-    <joint name="left_wheel_joint" type="continuous">
+    <joint name="right_wheel_joint" type="continuous">
         <parent link="origin_link"/>
-        <child link="left_wheel"/>
+        <child link="right_wheel"/>
         <!-- rotate wheel 90 deg around x-axis -->
         <origin xyz="0 -0.107 0" rpy="-${pi/2} 0 0"/>
@@ -143,12 +143,12 @@
     </joint>
     <!-- Right Wheel -->
-    <joint name="right_wheel_joint" type="continuous">
+    <joint name="left_wheel_joint" type="continuous">
         <parent link="origin_link"/>
-        <child link="right_wheel"/>
+        <child link="left_wheel"/>
         <origin xyz="0 0.107 0" rpy="${pi/2} 0 0"/>
         <axis xyz="0 0 -1"/>
     </joint>
     <!-- Front Passive Wheel -->
-    <joint name="front_passive_wheel_joint" type="continuous">
+    <joint name="front_passive_wheel_joint" type="fixed">
         <parent link="origin_link"/>
         <child link="front_passive_wheel"/>
@@ -156,5 +156,5 @@
     </joint>
     <!-- Back Passive Wheel -->
-    <joint name="back_passive_wheel_joint" type="continuous">
+    <joint name="back_passive_wheel_joint" type="fixed">
         <parent link="origin_link"/>
         <child link="back_passive_wheel"/>
